File: hardware/Segger-Breakout.kicad_sch (KiCad schematic)
At the start: 11 parts, among them J1 ESP32Pro Breakout2, J2 ESP32Pro Breakout1, J3 Pin Header Breakout, J4 JTag Segger Connector, J5 Rpi Pico Breakout1, J6 Rpi Pico Breakout2, P1 JTAG SWD Connector, U1 ProS3, U2 Rpi Pico

Commit message: schematic updates
Parts:
- removed J3: Pin Header Breakout, symbol hecatron.conn:JTAG_Segger_Connector
- added J7: Segger 5V Out, Connector_PinHeader_2.54mm:PinHeader_1x02_P2.54mm_Vertical, symbol Connector_Generic:Conn_01x02
- added J8: Segger Breakout, Connector_PinHeader_2.54mm:PinHeader_1x10_P2.54mm_Vertical, symbol Connector_Generic:Conn_01x10
- J1, J2: footprint (none) -> Connector_PinHeader_2.54mm:PinHeader_1x17_P2.54mm_Vertical
- J4: footprint (none) -> Connector_IDC:IDC-Header_2x10_P2.54mm_Vertical
- J5, J6: footprint (none) -> Connector_PinHeader_2.54mm:PinHeader_1x20_P2.54mm_Vertical
- JP1, JP2: footprint (none) -> Connector_PinSocket_2.54mm:PinSocket_1x02_P2.54mm_Vertical
- P1: footprint (none) -> hecatron.smd:ARM_10_PIN
- U1: footprint (none) -> pros3:ProS3_TH
- U2: footprint RPi_Pico:RPi_Pico_SMD_TH -> MCU_RaspberryPi_and_Boards:RPi_PicoW_SMD_TH
Connections:
- net +5V: now also J7.1 (Pin_1)
- net GND: now also J7.2 (Pin_2), J8.10 (Pin_10)
- net JTAG.DBGRQ: now also J8.9 (Pin_9)
- net JTAG.RESET: now also J8.8 (Pin_8)
- net JTAG.RTCK: now also J8.6 (Pin_6)
- net JTAG.TCK: now also J8.5 (Pin_5)
- net JTAG.TDI: now also J8.3 (Pin_3)
- net JTAG.TDO: now also J8.7 (Pin_7)
- net JTAG.TMS: now also J8.4 (Pin_4)
- net JTAG.~{nTRST}: now also J8.2 (Pin_2)
- net at J1.4 (Pin_4), U1.4 (3V3): now also JP1.1 (A); no longer JP1.2 (B)
- net at J6.5 (Pin_5), U2.36 (3V3): now also JP2.1 (A); no longer JP2.2 (B)
- net VCC renamed JTAG.VTRef
- net JTAG.VTRef: now also JP1.2 (B), JP2.2 (B), J8.1 (Pin_1); no longer JP1.1 (A), JP2.1 (A)
Other:
- moved on the sheet: JP1, JP2

Commit message: pcb updates
Parts:
- JP1, JP2: value VCC (USB Disconnected) -> VTref Segger Input
Changed lines of the file:
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@@
     (effects (font (size 1.27 1.27)) (justify right bottom))
   )
-  (label "JTAG.VTRef" (at 40.64 39.37 180)
+  (label "JTAG.VTRef" (at 40.64 39.37 180) (fields_autoplaced)
     (effects (font (size 1.27 1.27)) (justify right bottom))
   )
@@
       (effects (font (size 1.27 1.27)))
     )
-    (property "Value" "VCC (USB Disconnected)" (at 182.88 57.15 0)
+    (property "Value" "VTref Segger Input" (at 182.88 57.15 0)
       (effects (font (size 1.27 1.27)) hide)
     )
@@
       (effects (font (size 1.27 1.27)))
     )
-    (property "Value" "VCC (USB Disconnected)" (at 255.27 81.28 0)
-      (effects (font (size 1.27 1.27)) hide)
-    )
+    (property "Value" "VTref Segger Input" (at 255.27 81.28 0)
+      (effects (font (size 1.27 1.27)) hide)
+    )
